File: Open_hand/Open_hand.kicad_pcb (KiCad board)
At the start: 2 copper layers, 146.1 x 190 mm, 23 parts

Commit message: update
Parts:
- removed REF** (x19): LGA-14_3x2.5mm_P0.5mm_LayoutBorder3x4y, Package_LGA:LGA-14_3x2.5mm_P0.5mm_LayoutBorder3x4y
- removed REF**: ESP32-S3-WROOM-1, RF_Module:ESP32-S3-WROOM-1
- removed REF**: QFN-56-1EP_7x7mm_P0.4mm_EP3.2x3.2mm, Package_DFN_QFN:QFN-56-1EP_7x7mm_P0.4mm_EP3.2x3.2mm
- removed REF**: USB_C_Receptacle_HRO_TYPE-C-31-M-12, Connector_USB:USB_C_Receptacle_HRO_TYPE-C-31-M-12
- removed REF**: SOIC-8_3.9x4.9mm_P1.27mm, Package_SO:SOIC-8_3.9x4.9mm_P1.27mm
- added C10: 100n, Capacitor_SMD:C_0603_1608Metric, F.Cu at (174.9, 35.7)
- added C11: 10n, Capacitor_SMD:C_0402_1005Metric, F.Cu at (170.3, 37.8)
- added C12: 2u2, Capacitor_SMD:C_0603_1608Metric, F.Cu at (213.6, 161.8)
- added C13: 100n, Capacitor_SMD:C_0603_1608Metric, F.Cu at (213.6, 164.3)
- added C14: 10n, Capacitor_SMD:C_0402_1005Metric, F.Cu at (217.1, 165.6)
- added C15: 2u2, Capacitor_SMD:C_0603_1608Metric, F.Cu at (224.2, 137.8)
- added C16: 100n, Capacitor_SMD:C_0603_1608Metric, F.Cu at (224.2, 140.3)
- added C17: 10n, Capacitor_SMD:C_0402_1005Metric, F.Cu at (227.6, 141.5)
- added C18: 2u2, Capacitor_SMD:C_0603_1608Metric, F.Cu at (224.2, 161.8)
- added C19: 100n, Capacitor_SMD:C_0603_1608Metric, F.Cu at (224.2, 164.3)
- added C20: 10n, Capacitor_SMD:C_0402_1005Metric, F.Cu at (227.6, 165.6)
- added C21: 2u2, Capacitor_SMD:C_0603_1608Metric, F.Cu at (203.1, 137.8)
- added C22: 100n, Capacitor_SMD:C_0603_1608Metric, F.Cu at (203.1, 140.3)
- added C23: 10n, Capacitor_SMD:C_0402_1005Metric, F.Cu at (206.5, 141.5)
- added C24: 2u2, Capacitor_SMD:C_0603_1608Metric, F.Cu at (203.1, 169.8)
- added C25: 100n, Capacitor_SMD:C_0603_1608Metric, F.Cu at (203.1, 172.3)
- added C26: 10n, Capacitor_SMD:C_0402_1005Metric, F.Cu at (206.5, 173.6)
- added C27: 2u2, Capacitor_SMD:C_0603_1608Metric, F.Cu at (224.2, 145.8)
- added C28: 100n, Capacitor_SMD:C_0603_1608Metric, F.Cu at (224.2, 148.3)
- added C29: 10n, Capacitor_SMD:C_0402_1005Metric, F.Cu at (227.6, 149.6)
- added C3: 2u2, Capacitor_SMD:C_0603_1608Metric, F.Cu at (174.9, 101.5)
- added C30: 2u2, Capacitor_SMD:C_0603_1608Metric, F.Cu at (213.6, 145.8)
- added C31: 100n, Capacitor_SMD:C_0603_1608Metric, F.Cu at (213.6, 148.3)
- added C32: 10n, Capacitor_SMD:C_0402_1005Metric, F.Cu at (217.1, 149.6)
- added C33: 2u2, Capacitor_SMD:C_0603_1608Metric, F.Cu at (203.1, 161.8)
- added C34: 100n, Capacitor_SMD:C_0603_1608Metric, F.Cu at (203.1, 164.3)
- added C35: 10n, Capacitor_SMD:C_0402_1005Metric, F.Cu at (206.5, 165.6)
- added C36: 2u2, Capacitor_SMD:C_0603_1608Metric, F.Cu at (224.2, 153.8)
- added C37: 100n, Capacitor_SMD:C_0603_1608Metric, F.Cu at (224.2, 156.3)
- added C38: 10n, Capacitor_SMD:C_0402_1005Metric, F.Cu at (227.6, 157.6)
- added C39: 2u2, Capacitor_SMD:C_0603_1608Metric, F.Cu at (203.1, 153.8)
- added C4: 100n, Capacitor_SMD:C_0603_1608Metric, F.Cu at (173.3, 101.5)
- added C40: 100n, Capacitor_SMD:C_0603_1608Metric, F.Cu at (203.1, 156.3)
- added C41: 10n, Capacitor_SMD:C_0402_1005Metric, F.Cu at (206.5, 157.6)
- added C42: 2u2, Capacitor_SMD:C_0603_1608Metric, F.Cu at (203.1, 145.8)
- added C43: 100n, Capacitor_SMD:C_0603_1608Metric, F.Cu at (203.1, 148.3)
- added C44: 10n, Capacitor_SMD:C_0402_1005Metric, F.Cu at (206.5, 149.6)
- added C45: 2u2, Capacitor_SMD:C_0603_1608Metric, F.Cu at (213.6, 153.8)
- added C46: 100n, Capacitor_SMD:C_0603_1608Metric, F.Cu at (213.6, 156.3)
- added C47: 10n, Capacitor_SMD:C_0402_1005Metric, F.Cu at (217.1, 157.6)
- added C48: 2u2, Capacitor_SMD:C_0603_1608Metric, F.Cu at (176.9, 144.5)
- added C49: 100n, Capacitor_SMD:C_0603_1608Metric, F.Cu at (176.9, 147.0)
- added C5: 10n, Capacitor_SMD:C_0402_1005Metric, F.Cu at (170.3, 103.7)
- added C50: 10n, Capacitor_SMD:C_0402_1005Metric, F.Cu at (180.4, 148.3)
- added C51: 2u2, Capacitor_SMD:C_0603_1608Metric, F.Cu at (176.9, 152.5)
- added C52: 100n, Capacitor_SMD:C_0603_1608Metric, F.Cu at (176.9, 155.1)
- added C53: 10n, Capacitor_SMD:C_0402_1005Metric, F.Cu at (180.4, 156.3)
- added C54: 2u2, Capacitor_SMD:C_0603_1608Metric, F.Cu at (187.5, 144.5)
- added C55: 100n, Capacitor_SMD:C_0603_1608Metric, F.Cu at (187.5, 147.0)
- added C56: 10n, Capacitor_SMD:C_0402_1005Metric, F.Cu at (190.9, 148.3)
- added C6: 2u2, Capacitor_SMD:C_0603_1608Metric, F.Cu at (173.3, 67.3)
- added C7: 100n, Capacitor_SMD:C_0603_1608Metric, F.Cu at (174.9, 67.3)
- added C8: 10n, Capacitor_SMD:C_0402_1005Metric, F.Cu at (170.3, 69.5)
- added C9: 2u2, Capacitor_SMD:C_0603_1608Metric, F.Cu at (173.3, 35.7)
- added J1: USB_C_Receptacle_USB2.0, Connector_USB:USB_C_Receptacle_HRO_TYPE-C-31-M-12, F.Cu at (215.0, 212.0)
- added J2: USB_A, Connector_USB:USB_A_TE_292303-7_Horizontal, F.Cu at (198.0, 208.0)
- added U1: FUSB302B10MPX, Package_DFN_QFN:WQFN-14-1EP_2.5x2.5mm_P0.5mm_EP1.45x1.45mm, F.Cu at (212.0, 199.0)
- added U10: ICM-40608, Package_LGA:LGA-14_3x2.5mm_P0.5mm_LayoutBorder3x4y, F.Cu at (207.3, 138.5)
- added U11: ICM-40608, Package_LGA:LGA-14_3x2.5mm_P0.5mm_LayoutBorder3x4y, F.Cu at (207.3, 170.6)
- added U12: ICM-40608, Package_LGA:LGA-14_3x2.5mm_P0.5mm_LayoutBorder3x4y, F.Cu at (228.5, 146.6)
- added U13: ICM-40608, Package_LGA:LGA-14_3x2.5mm_P0.5mm_LayoutBorder3x4y, F.Cu at (217.9, 146.6)
- added U14: ICM-40608, Package_LGA:LGA-14_3x2.5mm_P0.5mm_LayoutBorder3x4y, F.Cu at (207.3, 162.6)
- added U15: ICM-40608, Package_LGA:LGA-14_3x2.5mm_P0.5mm_LayoutBorder3x4y, F.Cu at (228.5, 154.6)
- added U16: ICM-40608, Package_LGA:LGA-14_3x2.5mm_P0.5mm_LayoutBorder3x4y, F.Cu at (207.3, 154.6)
- added U17: ICM-40608, Package_LGA:LGA-14_3x2.5mm_P0.5mm_LayoutBorder3x4y, F.Cu at (207.3, 146.6)
- added U18: ICM-40608, Package_LGA:LGA-14_3x2.5mm_P0.5mm_LayoutBorder3x4y, F.Cu at (217.9, 154.6)
- added U19: ICM-40608, Package_LGA:LGA-14_3x2.5mm_P0.5mm_LayoutBorder3x4y, F.Cu at (181.2, 145.3)
- added U2: W25Q16JVSS, Package_SO:SOIC-8_5.23x5.23mm_P1.27mm, F.Cu at (224.0, 198.0)
- added U20: ICM-40608, Package_LGA:LGA-14_3x2.5mm_P0.5mm_LayoutBorder3x4y, F.Cu at (181.2, 153.3)
- added U21: ICM-40608, Package_LGA:LGA-14_3x2.5mm_P0.5mm_LayoutBorder3x4y, F.Cu at (191.8, 145.3)
- added U3: RP2040, Package_DFN_QFN:QFN-56-1EP_7x7mm_P0.4mm_EP3.2x3.2mm, F.Cu at (216.0, 189.0)
- added U4: ICM-40608, Package_LGA:LGA-14_3x2.5mm_P0.5mm_LayoutBorder3x4y, F.Cu at (170.5, 101.5)
- added U5: ICM-40608, Package_LGA:LGA-14_3x2.5mm_P0.5mm_LayoutBorder3x4y, F.Cu at (170.5, 67.3)
- added U6: ICM-40608, Package_LGA:LGA-14_3x2.5mm_P0.5mm_LayoutBorder3x4y, F.Cu at (170.5, 35.7)
- added U7: ICM-40608, Package_LGA:LGA-14_3x2.5mm_P0.5mm_LayoutBorder3x4y, F.Cu at (217.9, 162.6)
- added U8: ICM-40608, Package_LGA:LGA-14_3x2.5mm_P0.5mm_LayoutBorder3x4y, F.Cu at (228.5, 138.5)
- added U9: ICM-40608, Package_LGA:LGA-14_3x2.5mm_P0.5mm_LayoutBorder3x4y, F.Cu at (228.5, 162.6)
Routing:
- net /DOUT: track 0.00 -> 70.0 mm, vias 0 -> 3
- net /CLK: track 0.00 -> 69.4 mm, vias 0 -> 3
- net /DIN: track 0.00 -> 69.2 mm, vias 0 -> 3
- net GND: track 0.00 -> 19.4 mm
- net +3.3V: track 0.00 -> 13.7 mm
- net Net-(U2-IO2): track 0.00 -> 8.37 mm
- net Net-(U2-DO(IO1)): track 0.00 -> 7.03 mm
- net Net-(U2-~{CS}): track 0.00 -> 5.23 mm
- added copper zone on B.Cu, net GND
- added copper zone on F.Cu, net GND
- removed copper zone on B.Cu, net (none)
- removed copper zone on F.Cu, net (none)
Other:
- board text added: "0.0800 mm / 0.0800 mm"
- board text added: "0.1100 mm"
- board text added: "0.2500 mm"
- board text added: "146.0746 mm x 190.0000 mm"
- board text added: "2"
- board text added: "BOARD CHARACTERISTICS"
- board text added: "Board Thickness:"
- board text added: "Board overall dimensions:"
- board text added: "Castellated pads:"
- board text added: "Copper Finish:"
- board text added: "Copper Layer Count:"
- board text added: "Edge card connectors:"
- board text added: "Impedance Control:"
- board text added: "Min hole diameter:"
- board text added: "Min track/spacing:"
- board text added: "No"
- board text added: "None"
- board text added: "Plated Board Edge:"
- board text added: "Yes"
