File: Open_hand/Open_hand.kicad_sch (KiCad schematic)
At the start: 0 parts

Commit message: update
Changed lines of the file:
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@@
     )
   )
-  (sheet (at 74.93 48.895) (size 24.765 36.83) (fields_autoplaced)
+  (sheet (at 60.325 12.7) (size 24.765 36.83) (fields_autoplaced)
     (stroke (width 0.1524) (type solid))
     (fill (color 0 0 0 0.0000))
-    (property "Sheetname" "CPU" (at 74.93 48.1834 0)
+    (property "Sheetname" "CPU" (at 60.325 11.9884 0)
       (effects (font (size 1.27 1.27)) (justify left bottom))
     )
-    (property "Sheetfile" "CPU.kicad_sch" (at 74.93 86.3096 0)
+    (property "Sheetfile" "CPU.kicad_sch" (at 60.325 50.1146 0)
       (effects (font (size 1.27 1.27)) (justify left top))
     )
-    (property "Field2" "" (at 74.93 48.895 0)
+    (property "Field2" "" (at 60.325 12.7 0)
       (effects (font (size 1.27 1.27)) hide)
     )
