File: Open_hand_One_Finger/IMU.kicad_sch (KiCad schematic)
At the start: 4 parts, among them U5 ICM-40608

Commit message: add swd conector
Parts:
- renumbered C6 to C3, C7 to C4, C8 to C5, U5 to U4
Changed lines of the file:
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@@
   (symbol (lib_id "power:GND") (at 140.335 76.835 0) (unit 1)
     (in_bom yes) (on_board yes) (dnp no) (fields_autoplaced)
-    (property "Reference" "#PWR022" (at 140.335 83.185 0)
+    (property "Reference" "#PWR016" (at 140.335 83.185 0)
       (effects (font (size 1.27 1.27)) hide)
     )
@@
     (instances
       (project "Open_hand"
+        (path "/528d8ed7-b83e-40f9-82c3-8267528d108b/e2bb258b-f78d-4c92-a919-0a7042cdcd26"
+          (reference "#PWR016") (unit 1)
+        )
         (path "/528d8ed7-b83e-40f9-82c3-8267528d108b/f45c3bb1-fb6d-4b4c-94a8-5b9321358f13"
           (reference "#PWR022") (unit 1)
@@
           (reference "#PWR028") (unit 1)
         )
-        (path "/528d8ed7-b83e-40f9-82c3-8267528d108b/e2bb258b-f78d-4c92-a919-0a7042cdcd26"
-          (reference "#PWR016") (unit 1)
-        )
       )
     )
@@
   (symbol (lib_id "power:GND") (at 132.08 113.665 0) (unit 1)
     (in_bom yes) (on_board yes) (dnp no) (fields_autoplaced)
-    (property "Reference" "#PWR024" (at 132.08 120.015 0)
+    (property "Reference" "#PWR018" (at 132.08 120.015 0)
       (effects (font (size 1.27 1.27)) hide)
     )
@@
     (instances
       (project "Open_hand"
+        (path "/528d8ed7-b83e-40f9-82c3-8267528d108b/e2bb258b-f78d-4c92-a919-0a7042cdcd26"
+          (reference "#PWR018") (unit 1)
+        )
         (path "/528d8ed7-b83e-40f9-82c3-8267528d108b/f45c3bb1-fb6d-4b4c-94a8-5b9321358f13"
           (reference "#PWR024") (unit 1)
@@
           (reference "#PWR030") (unit 1)
         )
-        (path "/528d8ed7-b83e-40f9-82c3-8267528d108b/e2bb258b-f78d-4c92-a919-0a7042cdcd26"
-          (reference "#PWR018") (unit 1)
-        )
       )
     )
@@
   (symbol (lib_id "Device:C") (at 113.665 71.12 0) (unit 1)
     (in_bom yes) (on_board yes) (dnp no) (fields_autoplaced)
-    (property "Reference" "C6" (at 117.475 70.485 0)
+    (property "Reference" "C3" (at 117.475 70.485 0)
       (effects (font (size 1.27 1.27)) (justify left))
     )
@@
     (instances
       (project "Open_hand"
+        (path "/528d8ed7-b83e-40f9-82c3-8267528d108b/e2bb258b-f78d-4c92-a919-0a7042cdcd26"
+          (reference "C3") (unit 1)
+        )
         (path "/528d8ed7-b83e-40f9-82c3-8267528d108b/f45c3bb1-fb6d-4b4c-94a8-5b9321358f13"
           (reference "C6") (unit 1)
@@
           (reference "C9") (unit 1)
         )
-        (path "/528d8ed7-b83e-40f9-82c3-8267528d108b/e2bb258b-f78d-4c92-a919-0a7042cdcd26"
-          (reference "C3") (unit 1)
-        )
       )
     )
@@
   (symbol (lib_id "power:GND") (at 123.19 76.835 0) (unit 1)
     (in_bom yes) (on_board yes) (dnp no) (fields_autoplaced)
-    (property "Reference" "#PWR021" (at 123.19 83.185 0)
+    (property "Reference" "#PWR015" (at 123.19 83.185 0)
       (effects (font (size 1.27 1.27)) hide)
     )
@@
     (instances
       (project "Open_hand"
+        (path "/528d8ed7-b83e-40f9-82c3-8267528d108b/e2bb258b-f78d-4c92-a919-0a7042cdcd26"
+          (reference "#PWR015") (unit 1)
+        )
         (path "/528d8ed7-b83e-40f9-82c3-8267528d108b/f45c3bb1-fb6d-4b4c-94a8-5b9321358f13"
           (reference "#PWR021") (unit 1)
@@
           (reference "#PWR027") (unit 1)
         )
-        (path "/528d8ed7-b83e-40f9-82c3-8267528d108b/e2bb258b-f78d-4c92-a919-0a7042cdcd26"
-          (reference "#PWR015") (unit 1)
-        )
       )
     )
@@
   (symbol (lib_id "power:+3.3V") (at 133.35 62.23 0) (unit 1)
     (in_bom yes) (on_board yes) (dnp no) (fields_autoplaced)
-    (property "Reference" "#PWR019" (at 133.35 66.04 0)
+    (property "Reference" "#PWR013" (at 133.35 66.04 0)
       (effects (font (size 1.27 1.27)) hide)
     )
@@
     (instances
       (project "Open_hand"
+        (path "/528d8ed7-b83e-40f9-82c3-8267528d108b/e2bb258b-f78d-4c92-a919-0a7042cdcd26"
+          (reference "#PWR013") (unit 1)
+        )
         (path "/528d8ed7-b83e-40f9-82c3-8267528d108b/f45c3bb1-fb6d-4b4c-94a8-5b9321358f13"
           (reference "#PWR019") (unit 1)
@@
         (path "/528d8ed7-b83e-40f9-82c3-8267528d108b/2828d35a-0b94-4671-ad90-1bab511aff69"
           (reference "#PWR025") (unit 1)
-        )
-        (path "/528d8ed7-b83e-40f9-82c3-8267528d108b/e2bb258b-f78d-4c92-a919-0a7042cdcd26"
-          (reference "#PWR013") (unit 1)
         )
       )
@@
   (symbol (lib_id "IMU:ICM-40608") (at 120.65 72.39 0) (unit 1)
     (in_bom yes) (on_board yes) (dnp no)
-    (property "Reference" "U5" (at 134.0359 106.68 0)
+    (property "Reference" "U4" (at 134.0359 106.68 0)
       (effects (font (size 1.27 1.27)) (justify left))
     )
@@
     (instances
       (project "Open_hand"
+        (path "/528d8ed7-b83e-40f9-82c3-8267528d108b/e2bb258b-f78d-4c92-a919-0a7042cdcd26"
+          (reference "U4") (unit 1)
+        )
         (path "/528d8ed7-b83e-40f9-82c3-8267528d108b/f45c3bb1-fb6d-4b4c-94a8-5b9321358f13"
           (reference "U5") (unit 1)
@@
           (reference "U6") (unit 1)
         )
-        (path "/528d8ed7-b83e-40f9-82c3-8267528d108b/e2bb258b-f78d-4c92-a919-0a7042cdcd26"
-          (reference "U4") (unit 1)
-        )
       )
     )
@@
   (symbol (lib_id "Device:C") (at 140.335 71.12 0) (unit 1)
     (in_bom yes) (on_board yes) (dnp no) (fields_autoplaced)
-    (property "Reference" "C8" (at 144.145 70.485 0)
+    (property "Reference" "C5" (at 144.145 70.485 0)
       (effects (font (size 1.27 1.27)) (justify left))
     )
@@
     (instances
       (project "Open_hand"
+        (path "/528d8ed7-b83e-40f9-82c3-8267528d108b/e2bb258b-f78d-4c92-a919-0a7042cdcd26"
+          (reference "C5") (unit 1)
+        )
         (path "/528d8ed7-b83e-40f9-82c3-8267528d108b/f45c3bb1-fb6d-4b4c-94a8-5b9321358f13"
           (reference "C8") (unit 1)
@@
           (reference "C11") (unit 1)
         )
-        (path "/528d8ed7-b83e-40f9-82c3-8267528d108b/e2bb258b-f78d-4c92-a919-0a7042cdcd26"
-          (reference "C5") (unit 1)
-        )
       )
     )
@@
   (symbol (lib_id "power:GND") (at 119.38 113.665 0) (unit 1)
     (in_bom yes) (on_board yes) (dnp no) (fields_autoplaced)
-    (property "Reference" "#PWR023" (at 119.38 120.015 0)
+    (property "Reference" "#PWR017" (at 119.38 120.015 0)
       (effects (font (size 1.27 1.27)) hide)
     )
@@
     (instances
       (project "Open_hand"
+        (path "/528d8ed7-b83e-40f9-82c3-8267528d108b/e2bb258b-f78d-4c92-a919-0a7042cdcd26"
+          (reference "#PWR017") (unit 1)
+        )
         (path "/528d8ed7-b83e-40f9-82c3-8267528d108b/f45c3bb1-fb6d-4b4c-94a8-5b9321358f13"
           (reference "#PWR023") (unit 1)
@@
           (reference "#PWR029") (unit 1)
         )
-        (path "/528d8ed7-b83e-40f9-82c3-8267528d108b/e2bb258b-f78d-4c92-a919-0a7042cdcd26"
-          (reference "#PWR017") (unit 1)
-        )
       )
     )
@@
   (symbol (lib_id "Device:C") (at 123.19 71.12 0) (unit 1)
     (in_bom yes) (on_board yes) (dnp no) (fields_autoplaced)
-    (property "Reference" "C7" (at 127 70.485 0)
+    (property "Reference" "C4" (at 127 70.485 0)
       (effects (font (size 1.27 1.27)) (justify left))
     )
@@
     (instances
       (project "Open_hand"
+        (path "/528d8ed7-b83e-40f9-82c3-8267528d108b/e2bb258b-f78d-4c92-a919-0a7042cdcd26"
+          (reference "C4") (unit 1)
+        )
         (path "/528d8ed7-b83e-40f9-82c3-8267528d108b/f45c3bb1-fb6d-4b4c-94a8-5b9321358f13"
           (reference "C7") (unit 1)
@@
           (reference "C10") (unit 1)
         )
-        (path "/528d8ed7-b83e-40f9-82c3-8267528d108b/e2bb258b-f78d-4c92-a919-0a7042cdcd26"
-          (reference "C4") (unit 1)
-        )
       )
     )
@@
   (symbol (lib_id "power:GND") (at 113.665 76.835 0) (unit 1)
     (in_bom yes) (on_board yes) (dnp no) (fields_autoplaced)
-    (property "Reference" "#PWR020" (at 113.665 83.185 0)
+    (property "Reference" "#PWR014" (at 113.665 83.185 0)
       (effects (font (size 1.27 1.27)) hide)
     )
@@
     (instances
       (project "Open_hand"
+        (path "/528d8ed7-b83e-40f9-82c3-8267528d108b/e2bb258b-f78d-4c92-a919-0a7042cdcd26"
+          (reference "#PWR014") (unit 1)
+        )
         (path "/528d8ed7-b83e-40f9-82c3-8267528d108b/f45c3bb1-fb6d-4b4c-94a8-5b9321358f13"
           (reference "#PWR020") (unit 1)
@@
           (reference "#PWR026") (unit 1)
         )
-        (path "/528d8ed7-b83e-40f9-82c3-8267528d108b/e2bb258b-f78d-4c92-a919-0a7042cdcd26"
-          (reference "#PWR014") (unit 1)
-        )
-      )
+      )

Commit message: ajout des infos dans la cartouche
Other:
- title: (none) -> IMU schmatic for the Open Hand Project
Changed lines of the file:
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@@
 (kicad_sch (version 20230121) (generator eeschema)
   (paper "A4")
+  (title_block
+    (title "IMU schmatic for the Open Hand Project")
+    (date "2023-04-18")
+    (rev "Beta 1")
+    (comment 1 "Author : cdg66")
+  )
   (junction (at 123.19 62.23) (diameter 0) (color 0 0 0 0)
   )
