File: Open_hand_One_Finger/MAG.kicad_sch (KiCad schematic)
At the start: 6 parts, among them U1 LIS3MDL

Commit message: ajout des infos dans la cartouche
Other:
- title: (none) -> Magnetometer schmatic for the Open Hand Project
Changed lines of the file:
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@@
 (kicad_sch (version 20230121) (generator eeschema)
   (paper "A4")
+  (title_block
+    (title "Magnetometer schmatic for the Open Hand Project")
+    (date "2023-04-18")
+    (rev "Beta 1")
+    (comment 1 "Author : cdg66")
+  )
   (junction (at 142.875 58.42) (diameter 0) (color 0 0 0 0)
   )
